Commit message: Added optical camera link in .xacro

File: src/my_robot/urdf/my_robot.xacro (robot description, xacro)
@@ -180,4 +180,11 @@
 	  <parent link="chassis"/>
    </joint>
+  <joint name="camera_optical_joint" type="fixed">
+    <origin xyz="0 0 0" rpy="-1.5707 0 -1.5707"/>
+    <parent link="camera_link"/>
+    <child link="camera_link_optical"/>
+  </joint>
+  <link name="camera_link_optical">
+  </link>
   <gazebo reference="left_wheel">
     <material>Gazebo/Black</material>

Commit message: Naming the camera link properly

File: src/my_robot/urdf/my_robot.xacro (robot description, xacro)
@@ -182,5 +182,5 @@
   <joint name="camera_optical_joint" type="fixed">
     <origin xyz="0 0 0" rpy="-1.5707 0 -1.5707"/>
-    <parent link="camera_link"/>
+    <parent link="camera"/>
     <child link="camera_link_optical"/>
   </joint>
